Commit message: working! Though the walker is the wrong color and its cylinders instead of capsules

File: mpc_rl/tasks/walker/walker_modified.urdf (robot description, URDF)
Before this commit: robot converted_robot, 17 links, 16 joints
Links:
- link left_foot: geometry visual cylinder length=0.2 radius=0.05
- link left_leg: geometry visual cylinder length=0.5 radius=0.04
- link left_thigh: geometry visual cylinder length=0.45 radius=0.05
- link right_foot: geometry visual cylinder length=0.2 radius=0.05
- link right_leg: geometry visual cylinder length=0.5 radius=0.04
- link right_thigh: geometry visual cylinder length=0.45 radius=0.05
- link torso: geometry visual cylinder length=0.6 radius=0.07

Commit message: made the conversion script to make capsules (though kinda cheating via two spheres for each cylinder, but urdfs dont have capsules) and also made everything orange)

File: mpc_rl/tasks/walker/walker_modified.urdf (robot description, URDF)
Before this commit: robot converted_robot, 17 links, 16 joints
Links:
- link left_foot: geometry visual cylinder length=0.2 radius=0.05; visual sphere radius=0.05
- link left_leg: geometry visual cylinder length=0.5 radius=0.04; visual sphere radius=0.04
- link left_thigh: geometry visual cylinder length=0.45 radius=0.05; visual sphere radius=0.05
- link right_foot: geometry visual cylinder length=0.2 radius=0.05; visual sphere radius=0.05
- link right_leg: geometry visual cylinder length=0.5 radius=0.04; visual sphere radius=0.04
- link right_thigh: geometry visual cylinder length=0.45 radius=0.05; visual sphere radius=0.05
- link torso: geometry visual cylinder length=0.6 radius=0.07; visual sphere radius=0.07
